Commit message: with rviz

File: model/urdf/urdf.urdf (robot description, URDF)
Before this commit: robot urdf, 2 links, 1 joints
Links:
- added link base_link; visual cylinder length=0.1 radius=0.1
- link rod: mass 0.00785398163397448 -> None; geometry collision mesh filename=package://model/meshes/rod.STL; visual mesh filename=package://model/meshes/rod.STL
- link wheel_base: mass 0.029845130209103 -> None; geometry collision mesh filename=package://model/meshes/wheel_base.STL; visual mesh filename=package://model/meshes/wheel_base.STL
Joints:
- removed joint joint
- added joint base_to_wheel_x: type fixed, parent base_link, child wheel_base, origin xyz=0 0 0, axis 1 0 0, limit lower=-100 upper=100 effort=100 velocity=100
- added joint wheel_to_rod: type continuous, parent wheel_base, child rod, origin xyz=0 0 0 rpy=0 0 0, axis 0 -1 0
